File: kicad/sao_candle.kicad_pcb (KiCad board)
At the start: 2 copper layers, 22 x 44.1 mm, 12 parts, among them Q1 DMG2302U, X1 Simple_Addon_v2

Commit message: fixed documentation for read this time
Parts:
- R2: value 120 -> 100
