File: kicad/sao_candle.kicad_sch (KiCad schematic)
At the start: 12 parts, among them Q1 DMG2302U, X1 Simple_Addon_v2

Commit message: fixed documentation for read this time
Parts:
- R2: value 120 -> 100
Changed lines of the file:
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@@
 			)
 		)
-		(property "Value" "120"
+		(property "Value" "100"
 			(at 106.68 52.0699 0)
 			(show_name no)
